File: Sch/AMP-SPEAKER.sch (KiCad schematic (older format))
At the start: 31 parts, among them IC1 MCP4451-103E_ST, U2 PAM8403, U3 PAM8403

Commit message: Export netlist
Parts:
- removed U2: PAM8403, symbol v3-rescue:PAM8403-pam8403
- added U2: PAM8403, symbol PAM8403:PAM8403
- U3: symbol v3-rescue:PAM8403-pam8403 -> PAM8403:PAM8403
Connections:
- net GNDPWR: now also U2.15 (PGND), U2.2 (PGND)
- net TeensyGND: now also U2.11 (GND); no longer U3.9 (NC)
- net TeensyVDD: now also U2.6 (VDD)
- net at LS1.1: now also U2.1 (+OutLeft)
- net at R8.1: now also U2.10 (InRight)
- net at LS2.1: now also U2.14 (-OutRight)
- net at LS2.2: now also U2.16 (+OutRight)
- net at LS1.2: now also U2.3 (-OutLeft)
- net at R7.1: now also U2.7 (InLeft)
- net at C5.1: now also U2.8 (Vref)
- net +5V: no longer names the net of C10.2, C12.2, C14.2, U3.13 (PVDD), U3.4 (PVDD)
- net +5V: no longer C11.2, C13.2, C9.2
- new net: C11.2, C13.2, C9.2, U2.13 (PVDD), U2.4 (PVDD)
- no-connect marks 4 -> 5

Commit message: Update symbols and begin PCB
Parts:
- C1, C10, C11, C12, C13, C14, C2, C3, C4, C5, C6, C7, C8, C9: footprint (none) -> SMD Capacitor:CP_Elec_5x5.9
- IC1: footprint SOP65P640X120-20N -> MCP4451:SOP65P640X120-20N
- LS1, LS2, LS3, LS4: footprint (none) -> Pin Socket 2.54mm:PinSocket_2x02_P2.54mm_Vertical
- R1, R10, R2, R3, R4, R5, R6, R7, R8, R9: footprint (none) -> SMD Resistor:R_1218_3246Metric
- U2, U3: footprint (none) -> PAM8403:SOIC127P605X150-16N
