File: Sch/v3.sch (KiCad schematic (older format))
At the start: 1 part, among them U1 Teensy4.0

Commit message: Export netlist
Connections:
- net TeensyVDD: now also U1.31 (3V3); no longer U1.16 (3V3)
- net +BATT renamed +3V3
- net Freq1 renamed FREQ1
- net Freq10 renamed FREQ10
- net Freq11 renamed FREQ11
- net Freq12 renamed FREQ12
- net Freq13 renamed FREQ13
- net Freq14 renamed FREQ14
- net Freq15 renamed FREQ15
- net Freq16 renamed FREQ16
- net Freq2 renamed FREQ2
- net Freq3 renamed FREQ3
- net Freq4 renamed FREQ4
- net Freq5 renamed FREQ5
- net Freq6 renamed FREQ6
- net Freq7 renamed FREQ7
- net Freq8 renamed FREQ8
- net Freq9 renamed FREQ9
- net TeensySCL0 renamed SCL0
- net TeensySCL1 renamed SCL1
- net TeensySDA0 renamed SDA0
- net TeensySDA1 renamed SDA1
Changed lines of the file:
@@
 Text GLabel 3800 2350 0    50   Input ~ 0
 TeensyGND
-Text GLabel 3800 3850 0    50   Input ~ 0
-TeensyVDD
-Text GLabel 3800 4750 0    50   Input ~ 0
-TeensySDA0
-Text GLabel 3800 4850 0    50   Input ~ 0
-TeensySCL0
 Text GLabel 4900 5650 0    50   Input ~ 0
 TeensyGND
@@
 	0    -1   -1   0
 $EndComp
-Text GLabel 3800 4550 0    50   Input ~ 0
-TeensySCL1
-Text GLabel 3800 4650 0    50   Input ~ 0
-TeensySDA1
-Text GLabel 3800 2650 0    50   Input ~ 0
-Freq1
-Text GLabel 3800 2850 0    50   Input ~ 0
-Freq2
-Text GLabel 3800 2950 0    50   Input ~ 0
-Freq3
-Text GLabel 3800 3050 0    50   Input ~ 0
-Freq4
-Text GLabel 3800 3150 0    50   Input ~ 0
-Freq5
-Text GLabel 3800 3450 0    50   Input ~ 0
-Freq6
-Text GLabel 3800 3550 0    50   Input ~ 0
-Freq7
-Text GLabel 3800 3650 0    50   Input ~ 0
-Freq8
-Text GLabel 3800 4250 0    50   Input ~ 0
-Freq9
-Text GLabel 3800 4350 0    50   Input ~ 0
-Freq10
-Text GLabel 3800 4450 0    50   Input ~ 0
-Freq11
-Text GLabel 6200 5050 2    50   Input ~ 0
-Freq12
-Text GLabel 6200 3850 2    50   Input ~ 0
-Freq13
-Text GLabel 6200 3250 2    50   Input ~ 0
-Freq14
-Text GLabel 6200 2950 2    50   Input ~ 0
-Freq15
-Text GLabel 6200 2750 2    50   Input ~ 0
-Freq16
 Wire Wire Line
 	3800 2350 3900 2350
@@
 Wire Wire Line
 	3800 3650 3900 3650
-Wire Wire Line
-	3800 3850 3900 3850
 Wire Wire Line
 	3800 4250 3900 4250
@@
 $EndSheet
 $Comp
-L power:+BATT #PWR0101
+L power:+3.3V #PWR0101
 U 1 1 61A8BD0D
-P 6400 4650
-F 0 "#PWR0101" H 6400 4500 50  0001 C CNN
-F 1 "+BATT" H 6415 4823 50  0000 C CNN
-F 2 "" H 6400 4650 50  0001 C CNN
-F 3 "" H 6400 4650 50  0001 C CNN
-	1    6400 4650
+P 6200 4650
+F 0 "#PWR0101" H 6200 4500 50  0001 C CNN
+F 1 "+3.3V" H 6215 4823 50  0000 C CNN
+F 2 "" H 6200 4650 50  0001 C CNN
+F 3 "" H 6200 4650 50  0001 C CNN
+	1    6200 4650
 	0    1    1    0
 $EndComp
-Wire Wire Line
-	6100 4650 6400 4650
 NoConn ~ 3900 2450
 NoConn ~ 3900 2550
@@
 NoConn ~ 3900 5050
 NoConn ~ 6100 4950
-NoConn ~ 6100 4850
 NoConn ~ 6100 4750
 NoConn ~ 6100 4550
@@
 NoConn ~ 3900 3750
 NoConn ~ 3900 2750
+Text GLabel 3800 2650 0    50   Output ~ 0
+FREQ1
+Text GLabel 3800 2850 0    50   Output ~ 0
+FREQ2
+Text GLabel 3800 2950 0    50   Output ~ 0
+FREQ3
+Text GLabel 3800 3050 0    50   Output ~ 0
+FREQ4
+Text GLabel 3800 3150 0    50   Output ~ 0
+FREQ5
+Text GLabel 3800 3450 0    50   Output ~ 0
+FREQ6
+Text GLabel 3800 3550 0    50   Output ~ 0
+FREQ7
+Text GLabel 3800 3650 0    50   Output ~ 0
+FREQ8
+Text GLabel 6200 4850 2    50   Output ~ 0
+TeensyVDD
+Text GLabel 3800 4250 0    50   Output ~ 0
+FREQ9
+Text GLabel 3800 4350 0    50   Output ~ 0
+FREQ10
+Text GLabel 3800 4450 0    50   Output ~ 0
+FREQ11
+Text GLabel 3800 4550 0    50   BiDi ~ 0
+SCL1
+Text GLabel 3800 4650 0    50   BiDi ~ 0
+SDA1
+Text GLabel 3800 4750 0    50   BiDi ~ 0
+SDA0
+Text GLabel 3800 4850 0    50   BiDi ~ 0
+SCL0
+Text GLabel 6200 2750 2    50   Output ~ 0
+FREQ16
+Text GLabel 6200 2950 2    50   Output ~ 0
+FREQ15
+Text GLabel 6200 3250 2    50   Output ~ 0
+FREQ14
+Text GLabel 6200 3850 2    50   Output ~ 0
+FREQ13
+Text GLabel 6200 5050 2    50   Output ~ 0
+FREQ12
+NoConn ~ 3900 3850
+Wire Wire Line
+	6100 4850 6200 4850
+Wire Wire Line
+	6100 4650 6200 4650
+$Comp
+L power:PWR_FLAG #FLG0101
+U 1 1 60B5B8FC
+P 6200 4650
+F 0 "#FLG0101" H 6200 4725 50  0001 C CNN
+F 1 "PWR_FLAG" H 6200 4823 50  0000 C CNN
+F 2 "" H 6200 4650 50  0001 C CNN
+F 3 "~" H 6200 4650 50  0001 C CNN
+	1    6200 4650
+	1    0    0    -1
+$EndComp
+Connection ~ 6200 4650
 $EndSCHEMATC

Commit message: Update symbols and begin PCB
Parts:
- U1: footprint (none) -> Teensy:Teensy40_SMT
