File: AMP-SPEAKER.sch (KiCad schematic (older format))
At the start: 31 parts, among them IC1 MCP4451-103E_ST, U2 PAM8403, U3 PAM8403

Commit message: Some progress before reverting to 3/3 i2c line
Parts:
- removed C1, C2, C3, C4: 0.47uF, SMD Capacitor:CP_Elec_5x5.9, symbol v3-rescue:C-Device
- removed C10, C13, C14, C7, C8, C9: 1uF, SMD Capacitor:CP_Elec_5x5.9, symbol v3-rescue:C-Device
- removed C11, C12: 470uF, SMD Capacitor:CP_Elec_5x5.9, symbol v3-rescue:C-Device
- removed C5, C6: 0.1uF, SMD Capacitor:CP_Elec_5x5.9, symbol v3-rescue:C-Device
- removed R1, R2: 2200, SMD Resistor:R_1218_3246Metric, symbol v3-rescue:R-Device
- removed R10, R7, R8, R9: 10000, SMD Resistor:R_1218_3246Metric, symbol v3-rescue:R-Device
- removed U2, U3: PAM8403, PAM8403:SOIC127P605X150-16N, symbol PAM8403:PAM8403
- added U1, U14: AMPLIFIER-PAM8403, DIY modules:AMPLIFIER-PAM8403, symbol PAM8403-1:AMPLIFIER-PAM8403
- LS1, LS2, LS3, LS4: footprint Pin Socket 2.54mm:PinSocket_2x02_P2.54mm_Vertical -> Pin Socket 2.54mm:PinSocket_1x02_P2.54mm_Vertical
- R3, R4, R5, R6: footprint SMD Resistor:R_1218_3246Metric -> SMD Resistor:R_1206_3216Metric_Pad1.30x1.75mm_HandSolder
Connections:
- net labels added: A0, A1, GND, VDD
- net labels removed: GNDPWR
- wire segments 93 -> 50
- no-connect marks 5 -> 2

Commit message: Finalize PCB v0
Parts:
- renumbered R3 to R5, R4 to R6, R5 to R7, R6 to R8, U14 to U1, U1 to U2

Commit message: Release V3.0.1
Changed lines of the file:
@@
 $Descr A4 11693 8268
 encoding utf-8
-Sheet 5 7
+Sheet 2 7
 Title "Perception V3.0"
 Date "2021-05-10"
@@
 AR Path="/60B20965/60E20D4C" Ref="IC5"  Part="1"
 AR Path="/60B2096D/60E20D4C" Ref="IC6"  Part="1"
-F 0 "IC4" H 3700 3465 50  0001 C CNN
+F 0 "IC1" H 3700 3465 50  0001 C CNN
 F 1 "MCP4451-103E_ST" H 3700 3374 50  0000 C CNN
 F 2 "MCP4451:SOP65P640X120-20N" H 4200 3300 50  0001 L CNN
@@
 AR Path="/60B20965/60E20D7F" Ref="R21"  Part="1"
 AR Path="/60B2096D/60E20D7F" Ref="R25"  Part="1"
-F 0 "R17" V 2693 3200 50  0001 C CNN
+F 0 "R5" V 2693 3200 50  0001 C CNN
 F 1 "51000" V 2784 3200 50  0001 C CNN
 F 2 "SMD Resistor:R_1206_3216Metric_Pad1.30x1.75mm_HandSolder" V 2830 3200 50  0001 C CNN
@@
 AR Path="/60B20965/60E20D85" Ref="R22"  Part="1"
 AR Path="/60B2096D/60E20D85" Ref="R26"  Part="1"
-F 0 "R18" V 2693 4100 50  0001 C CNN
+F 0 "R6" V 2693 4100 50  0001 C CNN
 F 1 "51000" V 2784 4100 50  0001 C CNN
 F 2 "SMD Resistor:R_1206_3216Metric_Pad1.30x1.75mm_HandSolder" V 2830 4100 50  0001 C CNN
@@
 AR Path="/60B20965/60E20D8B" Ref="R24"  Part="1"
 AR Path="/60B2096D/60E20D8B" Ref="R28"  Part="1"
-F 0 "R20" V 4293 4100 50  0001 C CNN
+F 0 "R8" V 4293 4100 50  0001 C CNN
 F 1 "51000" V 4384 4100 50  0001 C CNN
 F 2 "SMD Resistor:R_1206_3216Metric_Pad1.30x1.75mm_HandSolder" V 4430 4100 50  0001 C CNN
@@
 AR Path="/60B20965/60E20D91" Ref="R23"  Part="1"
 AR Path="/60B2096D/60E20D91" Ref="R27"  Part="1"
-F 0 "R19" V 4293 3200 50  0001 C CNN
+F 0 "R7" V 4293 3200 50  0001 C CNN
 F 1 "51000" V 4384 3200 50  0001 C CNN
 F 2 "SMD Resistor:R_1206_3216Metric_Pad1.30x1.75mm_HandSolder" V 4430 3200 50  0001 C CNN
@@
 AR Path="/60B20965/60E20DA8" Ref="LS19"  Part="1"
 AR Path="/60B2096D/60E20DA8" Ref="LS23"  Part="1"
-F 0 "LS15" H 9720 2246 50  0000 L CNN
+F 0 "LS3" H 9720 2246 50  0000 L CNN
 F 1 "Speaker" H 9720 2155 50  0000 L CNN
 F 2 "Pin Socket 2.54mm:PinSocket_1x02_P2.54mm_Vertical" H 9550 2050 50  0001 C CNN
@@
 AR Path="/60B20965/60E20DAE" Ref="LS20"  Part="1"
 AR Path="/60B2096D/60E20DAE" Ref="LS24"  Part="1"
-F 0 "LS16" H 9720 2646 50  0000 L CNN
+F 0 "LS4" H 9720 2646 50  0000 L CNN
 F 1 "Speaker" H 9720 2555 50  0000 L CNN
 F 2 "Pin Socket 2.54mm:PinSocket_1x02_P2.54mm_Vertical" H 9550 2450 50  0001 C CNN
@@
 AR Path="/60B20965/60E20E32" Ref="LS17"  Part="1"
 AR Path="/60B2096D/60E20E32" Ref="LS21"  Part="1"
-F 0 "LS13" H 9670 4796 50  0000 L CNN
+F 0 "LS1" H 9670 4796 50  0000 L CNN
 F 1 "Speaker" H 9670 4705 50  0000 L CNN
 F 2 "Pin Socket 2.54mm:PinSocket_1x02_P2.54mm_Vertical" H 9500 4600 50  0001 C CNN
@@
 AR Path="/60B20965/60E20E38" Ref="LS18"  Part="1"
 AR Path="/60B2096D/60E20E38" Ref="LS22"  Part="1"
-F 0 "LS14" H 9670 5196 50  0000 L CNN
+F 0 "LS2" H 9670 5196 50  0000 L CNN
 F 1 "Speaker" H 9670 5105 50  0000 L CNN
 F 2 "Pin Socket 2.54mm:PinSocket_1x02_P2.54mm_Vertical" H 9500 5000 50  0001 C CNN
@@
 AR Path="/60B20965/60CD6CAD" Ref="U9"  Part="1"
 AR Path="/60B2096D/60CD6CAD" Ref="U11"  Part="1"
-F 0 "U7" H 7850 3117 50  0000 C CNN
+F 0 "U1" H 7850 3117 50  0000 C CNN
 F 1 "AMPLIFIER-PAM8403" H 7850 3026 50  0000 C CNN
 F 2 "DIY modules:AMPLIFIER-PAM8403" H 7850 2450 50  0001 L BNN
@@
 AR Path="/60B20965/60D0C2F9" Ref="U10"  Part="1"
 AR Path="/60B2096D/60D0C2F9" Ref="U12"  Part="1"
-F 0 "U8" H 7900 5667 50  0000 C CNN
+F 0 "U2" H 7900 5667 50  0000 C CNN
 F 1 "AMPLIFIER-PAM8403" H 7900 5576 50  0000 C CNN
 F 2 "DIY modules:AMPLIFIER-PAM8403" H 7900 5000 50  0001 L BNN
