File: V3.kicad_pcb (KiCad board)
At the start: 2 copper layers, 158 x 98.1 mm, 73 parts, among them IC1 MCP4451-103E_ST, IC2 MCP4451-103E_ST, IC3 MCP4451-103E_ST, IC4 MCP4451-103E_ST, IC5 MCP4451-103E_ST, IC6 MCP4451-103E_ST, J1 Conn_01x22_Female, J2 PowerPole, U1 AMPLIFIER-PAM8403, U10 AMPLIFIER-PAM8403, U11 AMPLIFIER-PAM8403, U12 AMPLIFIER-PAM8403, U2 AMPLIFIER-PAM8403, U3 AMPLIFIER-PAM8403, U4 AMPLIFIER-PAM8403, U5 AMPLIFIER-PAM8403, U6 AMPLIFIER-PAM8403, U7 AMPLIFIER-PAM8403, U8 AMPLIFIER-PAM8403, U9 AMPLIFIER-PAM8403

Commit message: Clean V3.0
Parts:
- removed ?: , HART:hart-logo-2000-2000dpi
- removed IC1, IC2, IC3, IC4, IC5, IC6: MCP4451-103E_ST, MCP4451:SOP65P640X120-20N
- removed J1: Conn_01x22_Female, Pin Socket 2.54mm:PinSocket_2x11_P2.54mm_Vertical
- removed J2: PowerPole, PowerPole:45A-VERT-PAIR
- removed LS1, LS10, LS11, LS12, LS13, LS14, LS15, LS16, LS17, LS18, LS19, LS2, LS20, LS21, LS22, LS23, LS24, LS3, LS4, LS5, LS6, LS7, LS8, LS9: Speaker, Pin Socket 2.54mm:PinSocket_1x02_P2.54mm_Vertical
- removed R1, R2, R3, R4: 2200, SMD Resistor:R_1206_3216Metric_Pad1.30x1.75mm_HandSolder
- removed R10, R11, R12, R13, R14, R15, R16, R17, R18, R19, R20, R21, R22, R23, R24, R25, R26, R27, R28, R5, R6, R7, R8, R9: 51000, SMD Resistor:R_1206_3216Metric_Pad1.30x1.75mm_HandSolder
- removed U1, U10, U11, U12, U2, U3, U4, U5, U6, U7, U8, U9: AMPLIFIER-PAM8403, DIY modules:AMPLIFIER-PAM8403
Routing:
- net GND: track 837.5 -> 0.00 mm, vias 3 -> 0
- net VDD: track 418.0 -> 0.00 mm
- net TeensyVDD: track 388.4 -> 0.00 mm, vias 15 -> 0
- net SCL1: track 214.8 -> 0.00 mm, vias 9 -> 0
- net SDA1: track 213.2 -> 0.00 mm, vias 7 -> 0
- net SCL0: track 181.2 -> 0.00 mm, vias 9 -> 0
- net SDA0: track 177.6 -> 0.00 mm, vias 7 -> 0
- net FREQ16: track 163.0 -> 0.00 mm, vias 3 -> 0
- net FREQ10: track 160.9 -> 0.00 mm, vias 3 -> 0
- net FREQ9: track 144.9 -> 0.00 mm, vias 3 -> 0
- net FREQ15: track 141.5 -> 0.00 mm, vias 3 -> 0
- net FREQ3: track 116.8 -> 0.00 mm, vias 3 -> 0
- net FREQ4: track 115.4 -> 0.00 mm, vias 3 -> 0
- net FREQ12: track 111.5 -> 0.00 mm, vias 3 -> 0
- net FREQ1: track 99.1 -> 0.00 mm, vias 3 -> 0
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Other:
- board outline removed
- copper layers 2 -> 4
- board text removed: "HARTware"
- board text removed: "Prototype V3"
