File: v3.sch (KiCad schematic (older format))
At the start: 1 part, among them U1 Teensy4.0

Commit message: Some progress before reverting to 3/3 i2c line
Parts:
- removed U1: Teensy4.0, Teensy:Teensy40_SMT, symbol teensy:Teensy4.0
- added J1: Barrel_Jack, Barrel Jack:BarrelJack_CUI_PJ-102AH_Horizontal, symbol Connector:Barrel_Jack
- added J2: Conn_01x22_Female, Pin Socket 2.54mm:PinSocket_2x11_P2.54mm_Vertical, symbol Connector:Conn_01x22_Female
- added R1, R2, R7, R8: 2200, SMD Resistor:R_1206_3216Metric_Pad1.30x1.75mm_HandSolder, symbol v3-rescue:R-Device
Connections:
- net labels added: +5V, GND, TeensyVVD, VDD
- net labels removed: +3.3V, GNDPWR
- wire segments 99 -> 133
- no-connect marks 31 -> 0

Commit message: Finalize PCB v0
Parts:
- renumbered R7 to R3, R8 to R4
Changed lines of the file:
@@
 $EndSheet
 $Sheet
-S 5650 4300 1600 850
+S 9000 900  1600 850
 U 60B2095D
 F0 "sheet60B20937" 50
 F1 "AMP-SPEAKER.sch" 50
-F2 "SCL" I L 5650 4650 50
-F3 "SDA" I L 5650 4800 50
-F4 "P1A" I L 5650 4450 50
-F5 "P0A" I L 5650 4350 50
-F6 "P2A" I L 5650 5000 50
-F7 "P3A" I L 5650 5100 50
-F8 "A0" I R 7250 4400 50
-F9 "A1" I R 7250 4500 50
+F2 "SCL" I L 9000 1250 50
+F3 "SDA" I L 9000 1400 50
+F4 "P1A" I L 9000 1050 50
+F5 "P0A" I L 9000 950 50
+F6 "P2A" I L 9000 1600 50
+F7 "P3A" I L 9000 1700 50
+F8 "A0" I R 10600 1000 50
+F9 "A1" I R 10600 1100 50
 $EndSheet
 $Sheet
@@
 Connection ~ 8200 3000
 Wire Wire Line
-	4500 4400 4750 4400
+	4500 3150 4750 3150
 Wire Wire Line
 	4750 1200 5650 1200
@@
 	4750 2350 4750 1200
 Wire Wire Line
-	4750 4650 5650 4650
-Wire Wire Line
 	5650 3500 4750 3500
-Connection ~ 4750 3500
-Wire Wire Line
-	4750 3500 4750 3950
-Wire Wire Line
-	4500 4550 4850 4550
-Wire Wire Line
-	4850 4800 5650 4800
+Wire Wire Line
+	4500 3300 4850 3300
 Wire Wire Line
 	5650 3650 4850 3650
-Connection ~ 4850 3650
 Wire Wire Line
 	5650 2500 4850 2500
@@
 Text GLabel 5550 3900 0    50   Input ~ 0
 FREQ10
-Text GLabel 5550 4400 0    50   Input ~ 0
+Text GLabel 8900 1000 0    50   Input ~ 0
 FREQ11
-Text GLabel 5550 5050 0    50   Input ~ 0
+Text GLabel 8900 1650 0    50   Input ~ 0
 FREQ12
 Wire Wire Line
@@
 	8200 3450 9000 3450
 Wire Wire Line
-	5600 5050 5600 5000
-Wire Wire Line
-	5600 5000 5650 5000
-Wire Wire Line
-	5550 5050 5600 5050
-Wire Wire Line
-	5600 5100 5600 5050
-Connection ~ 5600 5050
-Wire Wire Line
-	5600 5100 5650 5100
-Wire Wire Line
-	5550 4400 5600 4400
-Wire Wire Line
-	5600 4400 5600 4350
-Wire Wire Line
-	5600 4350 5650 4350
-Wire Wire Line
-	5650 4450 5600 4450
-Wire Wire Line
-	5600 4450 5600 4400
-Connection ~ 5600 4400
+	8950 1650 8950 1600
+Wire Wire Line
+	8950 1600 9000 1600
+Wire Wire Line
+	8900 1650 8950 1650
+Wire Wire Line
+	8950 1700 8950 1650
+Connection ~ 8950 1650
+Wire Wire Line
+	8950 1700 9000 1700
+Wire Wire Line
+	8900 1000 8950 1000
+Wire Wire Line
+	8950 1000 8950 950
+Wire Wire Line
+	8950 950  9000 950
+Wire Wire Line
+	9000 1050 8950 1050
+Wire Wire Line
+	8950 1050 8950 1000
+Connection ~ 8950 1000
 Wire Wire Line
 	5550 3900 5600 3900
@@
 Wire Wire Line
 	5550 900  5650 900
-Connection ~ 4750 4400
-Wire Wire Line
-	4750 4400 4750 4650
-Connection ~ 4850 4550
-Wire Wire Line
-	4850 4550 4850 4800
-Wire Wire Line
-	4750 2350 4750 3500
-Wire Wire Line
-	4850 2500 4850 3650
+Wire Wire Line
+	4750 2350 4750 2700
+Wire Wire Line
+	4850 2500 4850 2850
 Text GLabel 7350 1000 2    50   Input ~ 0
 TeensyGND
@@
 Text GLabel 7350 3250 2    50   Input ~ 0
 TeensyGND
-Text GLabel 10700 2100 2    50   Input ~ 0
-TeensyGND
-Text GLabel 10700 3300 2    50   Input ~ 0
+Text GLabel 10700 1050 2    50   Input ~ 0
+TeensyGND
+Text GLabel 10700 3200 2    50   Input ~ 0
 TeensyGND
 Wire Wire Line
@@
 Wire Wire Line
 	10600 3200 10700 3200
-Wire Wire Line
-	10600 2050 10650 2050
-Wire Wire Line
-	10650 2050 10650 2100
-Wire Wire Line
-	10650 2100 10700 2100
-Wire Wire Line
-	10600 2150 10650 2150
-Wire Wire Line
-	10650 2150 10650 2100
-Connection ~ 10650 2100
 Text GLabel 7350 2100 2    50   Input ~ 0
-TeensyVVD
+TeensyVDD
 Text GLabel 7350 3350 2    50   Input ~ 0
-TeensyVVD
-Text GLabel 7350 4450 2    50   Input ~ 0
-TeensyVVD
-Text GLabel 10700 3200 2    50   Input ~ 0
-TeensyVVD
+TeensyVDD
+Text GLabel 10700 3300 2    50   Input ~ 0
+TeensyVDD
 Wire Wire Line
 	10600 3300 10700 3300
@@
 	7250 3250 7350 3250
 Wire Wire Line
-	7250 4400 7300 4400
-Wire Wire Line
-	7300 4400 7300 4450
-Wire Wire Line
-	7300 4450 7350 4450
-Wire Wire Line
-	7250 4500 7300 4500
-Wire Wire Line
-	7300 4500 7300 4450
-Connection ~ 7300 4450
+	10600 1000 10650 1000
+Wire Wire Line
+	10650 1000 10650 1050
+Wire Wire Line
+	10650 1050 10700 1050
+Wire Wire Line
+	10600 1100 10650 1100
+Wire Wire Line
+	10650 1100 10650 1050
+Connection ~ 10650 1050
 Text GLabel 2850 2700 2    50   Output ~ 0
 FREQ8
@@
 Text GLabel 2850 3600 2    50   BiDi ~ 0
 SCL0
-Text GLabel 4500 4550 0    50   BiDi ~ 0
+Text GLabel 4500 3300 0    50   BiDi ~ 0
 SDA0
-Text GLabel 4500 4400 0    50   BiDi ~ 0
+Text GLabel 4500 3150 0    50   BiDi ~ 0
 SCL0
 Wire Wire Line
@@
 $EndComp
 $Comp
-L power:GND #PWR01
+L power:GND #PWR02
 U 1 1 60E483FB
 P 3900 1350
-F 0 "#PWR01" H 3900 1100 50  0001 C CNN
+F 0 "#PWR02" H 3900 1100 50  0001 C CNN
 F 1 "GND" H 3905 1177 50  0000 C CNN
 F 2 "" H 3900 1350 50  0001 C CNN
@@
 	3150 1000 3250 1000
 $Comp
-L power:+5V #PWR02
+L power:+5V #PWR01
 U 1 1 60E5F6BA
 P 2850 1000
-F 0 "#PWR02" H 2850 850 50  0001 C CNN
+F 0 "#PWR01" H 2850 850 50  0001 C CNN
 F 1 "+5V" H 2865 1173 50  0000 C CNN
 F 2 "" H 2850 1000 50  0001 C CNN
@@
 L v3-rescue:R-Device R2
 U 1 1 60C4431E
-P 4550 4100
+P 4550 2850
 AR Path="/60C4431E" Ref="R2"  Part="1"
 AR Path="/60B3C664/60C4431E" Ref="R?"  Part="1"
@@
 AR Path="/60B20965/60C4431E" Ref="R?"  Part="1"
 AR Path="/60B2096D/60C4431E" Ref="R?"  Part="1"
-F 0 "R2" V 4343 4100 50  0001 C CNN
-F 1 "2200" V 4434 4100 50  0001 C CNN
-F 2 "SMD Resistor:R_1206_3216Metric_Pad1.30x1.75mm_HandSolder" V 4480 4100 50  0001 C CNN
-F 3 "~" H 4550 4100 50  0001 C CNN
-	1    4550 4100
+F 0 "R2" V 4343 2850 50  0001 C CNN
+F 1 "2200" V 4434 2850 50  0001 C CNN
+F 2 "SMD Resistor:R_1206_3216Metric_Pad1.30x1.75mm_HandSolder" V 4480 2850 50  0001 C CNN
+F 3 "~" H 4550 2850 50  0001 C CNN
+	1    4550 2850
 	0    1    1    0
 $EndComp
@@
 L v3-rescue:R-Device R1
 U 1 1 60C44324
-P 4550 3950
+P 4550 2700
 AR Path="/60C44324" Ref="R1"  Part="1"
 AR Path="/60B3C664/60C44324" Ref="R?"  Part="1"
@@
 AR Path="/60B20965/60C44324" Ref="R?"  Part="1"
 AR Path="/60B2096D/60C44324" Ref="R?"  Part="1"
-F 0 "R1" V 4343 3950 50  0001 C CNN
-F 1 "2200" V 4434 3950 50  0001 C CNN
-F 2 "SMD Resistor:R_1206_3216Metric_Pad1.30x1.75mm_HandSolder" V 4480 3950 50  0001 C CNN
-F 3 "~" H 4550 3950 50  0001 C CNN
-	1    4550 3950
+F 0 "R1" V 4343 2700 50  0001 C CNN
+F 1 "2200" V 4434 2700 50  0001 C CNN
+F 2 "SMD Resistor:R_1206_3216Metric_Pad1.30x1.75mm_HandSolder" V 4480 2700 50  0001 C CNN
+F 3 "~" H 4550 2700 50  0001 C CNN
+	1    4550 2700
 	0    1    1    0
 $EndComp
-Text GLabel 4400 4100 0    50   Input ~ 0
-TeensyVDD
-Text GLabel 4400 3950 0    50   Input ~ 0
-TeensyVDD
-Wire Wire Line
-	4700 3950 4750 3950
-Connection ~ 4750 3950
-Wire Wire Line
-	4750 3950 4750 4400
-Wire Wire Line
-	4700 4100 4850 4100
-Wire Wire Line
-	4850 3650 4850 4100
-Connection ~ 4850 4100
-Wire Wire Line
-	4850 4100 4850 4550
-$Comp
-L v3-rescue:R-Device R8
+Text GLabel 4400 2850 0    50   Input ~ 0
+TeensyVDD
+Text GLabel 4400 2700 0    50   Input ~ 0
+TeensyVDD
+Wire Wire Line
+	4700 2700 4750 2700
+Wire Wire Line
+	4700 2850 4850 2850
+$Comp
+L v3-rescue:R-Device R4
 U 1 1 60C65139
 P 8000 2650
-AR Path="/60C65139" Ref="R8"  Part="1"
+AR Path="/60C65139" Ref="R4"  Part="1"
 AR Path="/60B3C664/60C65139" Ref="R?"  Part="1"
 AR Path="/60B3C664/60D625EB/60C65139" Ref="R?"  Part="1"
@@
 AR Path="/60B20965/60C65139" Ref="R?"  Part="1"
 AR Path="/60B2096D/60C65139" Ref="R?"  Part="1"
-F 0 "R8" V 7793 2650 50  0001 C CNN
+F 0 "R4" V 7793 2650 50  0001 C CNN
 F 1 "2200" V 7884 2650 50  0001 C CNN
 F 2 "SMD Resistor:R_1206_3216Metric_Pad1.30x1.75mm_HandSolder" V 7930 2650 50  0001 C CNN
@@
 $EndComp
 $Comp
-L v3-rescue:R-Device R7
+L v3-rescue:R-Device R3
 U 1 1 60C6513F
 P 8000 2500
-AR Path="/60C6513F" Ref="R7"  Part="1"
+AR Path="/60C6513F" Ref="R3"  Part="1"
 AR Path="/60B3C664/60C6513F" Ref="R?"  Part="1"
 AR Path="/60B3C664/60D625EB/60C6513F" Ref="R?"  Part="1"
@@
 AR Path="/60B20965/60C6513F" Ref="R?"  Part="1"
 AR Path="/60B2096D/60C6513F" Ref="R?"  Part="1"
-F 0 "R7" V 7793 2500 50  0001 C CNN
+F 0 "R3" V 7793 2500 50  0001 C CNN
 F 1 "2200" V 7884 2500 50  0001 C CNN
 F 2 "SMD Resistor:R_1206_3216Metric_Pad1.30x1.75mm_HandSolder" V 7930 2500 50  0001 C CNN
@@
 Wire Wire Line
 	8450 2650 8450 2450
+Connection ~ 4750 2700
+Wire Wire Line
+	4750 2700 4750 3150
+Connection ~ 4750 3150
+Wire Wire Line
+	4750 3150 4750 3500
+Connection ~ 4850 2850
+Wire Wire Line
+	4850 2850 4850 3300
+Connection ~ 4850 3300
+Wire Wire Line
+	4850 3300 4850 3650
+Text GLabel 10750 2150 2    50   Input ~ 0
+TeensyGND
+Text GLabel 10750 2050 2    50   Input ~ 0
+TeensyVDD
+Wire Wire Line
+	10600 2050 10750 2050
+Wire Wire Line
+	10600 2150 10750 2150
+Wire Wire Line
+	8450 2450 8450 1400
+Wire Wire Line
+	8450 1400 9000 1400
+Connection ~ 8450 2450
+Wire Wire Line
+	9000 1250 8200 1250
+Wire Wire Line
+	8200 1250 8200 2300
+Connection ~ 8200 2300
 $EndSCHEMATC

Commit message: Release V3.0.1
Parts:
- removed J1: Barrel_Jack, Barrel Jack:BarrelJack_CUI_PJ-102AH_Horizontal, symbol Connector:Barrel_Jack
- added J2: PowerPole, PowerPole:45A-VERT-PAIR, symbol AndersonPowerPole:PowerPole
- renumbered J2 to J1
Connections:
- net +5V: now also J2.1
- net GND: now also J2.2
Changed lines of the file:
@@
 	3900 1450 3900 1350
 $Comp
-L Connector:Conn_01x22_Female J2
+L Connector:Conn_01x22_Female J1
 U 1 1 60DEA836
 P 2550 2800
-F 0 "J2" H 2442 3985 50  0000 C CNN
+F 0 "J1" H 2442 3985 50  0000 C CNN
 F 1 "Conn_01x22_Female" H 2442 3894 50  0000 C CNN
 F 2 "Pin Socket 2.54mm:PinSocket_2x11_P2.54mm_Vertical" H 2550 2800 50  0001 C CNN
@@
 	1    2550 2800
 	-1   0    0    -1
-$EndComp
-$Comp
-L Connector:Barrel_Jack J1
-U 1 1 60E0F3C8
-P 2400 1100
-F 0 "J1" H 2457 1425 50  0000 C CNN
-F 1 "Barrel_Jack" H 2457 1334 50  0000 C CNN
-F 2 "Barrel Jack:BarrelJack_CUI_PJ-102AH_Horizontal" H 2450 1060 50  0001 C CNN
-F 3 "~" H 2450 1060 50  0001 C CNN
-	1    2400 1100
-	1    0    0    -1
 $EndComp
 $Comp
@@
 	8200 1250 8200 2300
 Connection ~ 8200 2300
+$Comp
+L AndersonPowerPole:PowerPole J2
+U 1 1 60DED7AA
+P 2400 850
+F 0 "J2" H 2457 925 50  0000 C CNN
+F 1 "PowerPole" H 2457 834 50  0000 C CNN
+F 2 "PowerPole:45A-VERT-PAIR" H 2400 850 50  0001 C CNN
+F 3 "" H 2400 850 50  0001 C CNN
+	1    2400 850
+	1    0    0    -1
+$EndComp
 $EndSCHEMATC
