File: V3-1-top.sch (KiCad schematic (older format))
At the start: 10 parts, among them J1 Conn_01x12_Female, J2 Conn_01x12_Female, J3 Conn_01x03_Male, J4 Conn_01x03_Male, J5 Conn_01x03_Male, J6 Conn_01x03_Male, J7 Conn_01x03_Male, J8 Conn_01x03_Male

Commit message: Done BOT v3.1
Connections:
- net GND: no longer J7.2 (Pin_2)
- no-connect marks 2 -> 3
Changed lines of the file:
@@
 Text GLabel 4550 1750 2    50   Input ~ 0
 FREQ16
-Text GLabel 4550 2600 2    50   Input ~ 0
-TeensyGND
 Text GLabel 4550 950  2    50   Input ~ 0
 VDD
@@
 Wire Notes Line
 	2850 550  2850 4600
+NoConn ~ 4550 2600
 $EndSCHEMATC

Commit message: Cleanup symbols and libraries and add separate submodule for kicad-libaries
Parts:
- R1, R2: symbol v3-rescue:R-Device -> pspice:R
Changed lines of the file:
@@
 Wire Wire Line
 	1250 1150 1350 1150
-Text GLabel 1600 4650 0    50   UnSpc ~ 0
+Text GLabel 1500 4650 0    50   UnSpc ~ 0
 TeensyVDD
 $Comp
-L v3-rescue:R-Device R1
+L pspice:R R1
 U 1 1 61323621
 P 1750 4650
@@
 	0    1    1    0
 $EndComp
-Text GLabel 1600 4800 0    50   UnSpc ~ 0
+Text GLabel 1500 4800 0    50   UnSpc ~ 0
 TeensyVDD
 $Comp
-L v3-rescue:R-Device R2
+L pspice:R R2
 U 1 1 61325776
 P 1750 4800
@@
 Text GLabel 2000 4650 2    50   Input ~ 0
 SDA1
-Wire Wire Line
-	1900 4800 2000 4800
-Wire Wire Line
-	1900 4650 2000 4650
 Text GLabel 2250 800  2    50   Output ~ 0
 SPEAK13-
